File: quaz_conn_part/quaz_conn_part.kicad_sch (KiCad schematic)
At the start: 6 parts

Commit message: next
Connections:
- net BT_OK: now also U?.40 (B11); no longer U?.1 (B12)
- net BT_ESC renamed BT_DOWN
- new net BT_UP: U?.1 (B12)
Changed lines of the file:
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@@
+    (stroke (width 0) (type default) (color 0 0 0 0))
+  )
+  (wire (pts (xy 127 59.69) (xy 139.7 59.69))
     (stroke (width 0) (type default) (color 0 0 0 0))
   )
@@
     (effects (font (size 1.27 1.27)) (justify right bottom))
   )
-  (label "BT_OK" (at 88.9 49.53 0)
+  (label "BT_UP" (at 88.9 49.53 0)
     (effects (font (size 1.27 1.27)) (justify left bottom))
   )
@@
     (effects (font (size 1.27 1.27)) (justify left bottom))
   )
-  (label "BT_ESC" (at 88.9 52.07 0)
+  (label "BT_DOWN" (at 88.9 52.07 0)
     (effects (font (size 1.27 1.27)) (justify left bottom))
   )
@@
     (effects (font (size 1.27 1.27)) (justify right bottom))
   )
+  (label "BT_OK" (at 139.7 59.69 180)
+    (effects (font (size 1.27 1.27)) (justify right bottom))
+  )
