File: quaz_conn_part/quaz_conn_part.kicad_sch (KiCad schematic)
At the start: 6 parts

Commit message: add some settings
Parts:
- added C? (x2): 0.1, symbol Device:C
- added R? (x2): 16K, symbol Device:R
- added R?: 10K, symbol Device:R
- added R?: 51K, symbol Device:R
Connections:
- net GND: now also C?.1, R?.2, R?.2
- net TX_I_SENS: now also C?.2; no longer U?.30 (A1)
- net ACC_SENS: now reaches U?.29 (A0)
- net ACC_SENS: now also C?.2, R?.1, R?.2
- net at U?.42 (3V3): now also R?.1
- new net: C?.1, R?.1, R?.2, U?.30 (A1)
- new net VPP: R?.1
