File: quaz_drv_part/quaz_drv_part.kicad_pcb (KiCad board)
At the start: 2 copper layers, 64.6 x 69.6 mm, 47 parts, among them J1 TX, J2 sound, J3 curs, J4 tx_src, J5 phones, J6 PWR, J7 speaker, J8 5Vout, J9 5Vout, U1 MC34119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

Commit message: drv layout change
Parts:
- C11: footprint Capacitor_THT:CP_Radial_D10.0mm_P5.00mm -> Capacitor_THT:CP_Radial_D8.0mm_P5.00mm
- C12, C18, D1, J6, J8, J9: moved to F.Cu
- C2: footprint Capacitor_THT:C_Disc_D9.0mm_W5.0mm_P5.00mm -> Capacitor_THT:C_Rect_L26.5mm_W7.0mm_P22.50mm_MKS4
- C3: footprint Capacitor_THT:C_Disc_D9.0mm_W5.0mm_P5.00mm -> Capacitor_THT:C_Rect_L11.0mm_W4.2mm_P10.00mm_MKT
- R2, R3: footprint Resistor_THT:R_Axial_Power_L20.0mm_W6.4mm_P7.62mm_Vertical -> Resistor_SMD:R_1218_3246Metric_Pad1.22x4.75mm_HandSolder; moved to F.Cu
- moved R8 173.2 mm to (214.4, 57.6)
- moved C8 171.1 mm to (214.4, 49.2), turned to 90 degrees
- moved J1 161.4 mm to (215.8, 69.7), turned to 0 degrees
- moved R7 161.1 mm to (204.8, 57.5), turned to 180 degrees
- moved U1 158.7 mm to (205.0, 51.0), turned to 0 degrees
- moved J7 155.8 mm to (187.9, 44.6), turned to -90 degrees
- moved C3 155.1 mm to (215.7, 75.5), turned to 180 degrees
- moved J5 155.0 mm to (203.2, 61.1), turned to 0 degrees
- moved C2 150.8 mm to (211.4, 68.7), turned to 180 degrees
- moved R5 148.9 mm to (198.9, 54.5), turned to -90 degrees
- moved JP1 142.8 mm to (178.9, 44.6), turned to -90 degrees
- moved C6 138.1 mm to (190.0, 57.9), turned to 90 degrees
- moved C4 137.8 mm to (180.4, 48.1), turned to 0 degrees
- moved J2 136.5 mm to (165.5, 44.4), turned to 180 degrees
- moved R1 136.2 mm to (186.0, 51.1), turned to 0 degrees
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Routing:
- net VCC: track 54.3 -> 5.24 mm
- net GND: track 0.00 -> 47.9 mm, vias 0 -> 2
- net Net-(C18-Pad1): track 28.6 -> 0.00 mm
- net Net-(JP1-Pad2): track 3.60 -> 23.0 mm
- net Net-(C4-Pad2): track 3.89 -> 22.0 mm
- net Net-(C6-Pad1): track 18.6 -> 34.2 mm, vias 0 -> 2
- net Net-(J1-Pad2): track 24.3 -> 39.4 mm
- net Net-(C10-Pad1): track 28.8 -> 14.9 mm
- net Net-(C8-Pad1): track 40.0 -> 53.5 mm
- net Net-(R7-Pad1): track 5.60 -> 14.2 mm, vias 0 -> 2
- net Net-(C22-Pad1): track 12.6 -> 6.44 mm
- net Net-(C2-Pad2): track 14.6 -> 20.3 mm
- net Net-(J5-PadRN): track 20.4 -> 24.9 mm
- net Net-(C6-Pad2): track 12.8 -> 16.6 mm
- net Net-(R2-Pad2): track 17.0 -> 20.5 mm
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- removed copper zone on F.Cu, net GND
Other:
- board outline removed

Commit message: add btn_part
Parts:
- C12, D1, J6, J8, J9: moved to B.Cu
- C18: footprint Capacitor_THT:CP_Radial_D10.0mm_P5.00mm -> Capacitor_THT:CP_Radial_D8.0mm_P5.00mm; moved to B.Cu
- moved C18 154.5 mm to (206.3, 86.3), turned to 90 degrees
- moved C12 131.9 mm to (197.1, 81.2), turned to 90 degrees
- moved J6 130.6 mm to (212.4, 80.1), turned to -90 degrees
- moved U5 126.7 mm to (191.6, 78.8), turned to -90 degrees
- moved J9 114.0 mm to (200.5, 88.4), turned to 90 degrees
- moved D1 107.5 mm to (179.5, 83.8), turned to 180 degrees
- moved J8 106.7 mm to (215.0, 86.8)
- moved U4 93.8 mm to (182.6, 77.9), turned to 180 degrees
- moved C16 86.3 mm to (178.1, 87.2), turned to 180 degrees
- moved C19 79.2 mm to (191.6, 87.5), turned to -90 degrees
- moved C13 78.7 mm to (200.1, 77.7), turned to 90 degrees
- moved C11 17.0 mm to (169.0, 85.7), turned to 180 degrees
- moved C4 14.0 mm to (194.3, 50.3)
Routing:
- net VCC: track 5.24 -> 109.0 mm, vias 0 -> 4
- net Net-(C18-Pad1): track 0.00 -> 36.7 mm
- net Net-(C10-Pad1): track 14.9 -> 32.0 mm
- net Net-(C4-Pad2): track 22.0 -> 7.27 mm
- net GND: track 47.9 -> 62.5 mm, vias 2 -> 4
- net Net-(C2-Pad2): track 20.3 -> 23.0 mm
- net Net-(R2-Pad2): track 20.5 -> 22.8 mm
- added copper zone on B.Cu, net GND
- added copper zone on F.Cu, net GND
Other:
- board outline added: 60.6 x 54.9 mm
