File: quaz_btn_part/quaz_btn_part.kicad_sch (KiCad schematic)
At the start: 2 parts

Commit message: add buttons board
Parts:
- added C1, C2, C3, C4, C5: 0.1, Capacitor_SMD:C_1206_3216Metric_Pad1.33x1.80mm_HandSolder, symbol Device:C
- added J1: Conn_01x07_Male, Connector_PinHeader_2.54mm:PinHeader_1x07_P2.54mm_Vertical, symbol Connector:Conn_01x07_Male
- added R1, R2, R3, R4, R5: 15K, Resistor_SMD:R_1206_3216Metric_Pad1.30x1.75mm_HandSolder, symbol Device:R
- added SW2: DOWN, quaz_btn_part:BTN13, symbol Switch:SW_DPDT_x2
- added SW3: INC, quaz_btn_part:BTN13, symbol Switch:SW_DPDT_x2
- added SW4: DEC, quaz_btn_part:BTN13, symbol Switch:SW_DPDT_x2
- added SW5: OK, quaz_btn_part:BTN13, symbol Switch:SW_DPDT_x2
- SW1: renamed from SW?; value SW_DPDT_x2 -> UP; footprint (none) -> quaz_btn_part:BTN13
Connections:
- net at SW1.2 (B): now also C1.1, J1.1 (Pin_1), R1.2
- net GND: now reaches SW1.3 (C)
- net GND: now also C1.2, C2.2, C3.2, C4.2, C5.2, J1.7 (Pin_7), SW2.3 (C), SW3.3 (C), SW4.3 (C), SW5.3 (C)
- new net: C2.1, J1.5 (Pin_5), R2.2, SW2.2 (B)
- new net: C4.1, J1.2 (Pin_2), R4.2, SW4.2 (B)
- new net: C3.1, J1.4 (Pin_4), R3.2, SW3.2 (B)
- new net: C5.1, J1.3 (Pin_3), R5.2, SW5.2 (B)
- new net +3V3: J1.6 (Pin_6), R1.1, R2.1, R3.1, R4.1, R5.1
- no-connect marks 0 -> 20
Other:
- moved on the sheet: SW1B
