File: quaz_btn_part/quaz_btn_part.kicad_pcb (KiCad board)
At the start: 2 copper layers, 52.5 x 38.2 mm, 16 parts, among them J1 Conn_01x07_Male, SW1 UP, SW2 DOWN, SW3 INC, SW4 DEC, SW5 OK

Commit message: pcb for buttons
Routing:
- net GND: track 52.3 -> 39.0 mm
- net Net-(J1-Pad1): track 31.0 -> 30.2 mm
- net (no net): vias 0 -> 4
Changed lines of the file:
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@@
     (pad_to_mask_clearance 0)
     (pcbplotparams
-      (layerselection 0x0001000_fffffffe)
+      (layerselection 0x0000000_fffffffe)
       (disableapertmacros false)
       (usegerberextensions false)
@@
       (psnegative false)
       (psa4output false)
-      (plotreference true)
-      (plotvalue true)
+      (plotreference false)
+      (plotvalue false)
       (plotinvisibletext false)
       (sketchpadsonfab false)
@@
   )
   (gr_rect (start 138.5 58.25) (end 191 96.5) (layer "Edge.Cuts") (width 0.1) (fill none))
+  (via (at 187 62.75) (size 4) (drill 3) (layers "F.Cu" "B.Cu") (free) (net 0))
+  (via (at 143 62.75) (size 4) (drill 3) (layers "F.Cu" "B.Cu") (free) (net 0))
+  (via (at 142.75 92) (size 4) (drill 3) (layers "F.Cu" "B.Cu") (free) (net 0))
+  (via (at 187 92.5) (size 4) (drill 3) (layers "F.Cu" "B.Cu") (free) (net 0))
   (via (at 173 90.75) (size 2.2) (drill 0.8) (layers "F.Cu" "B.Cu") (net 1))
   (via (at 145 84.5) (size 2.2) (drill 0.8) (layers "F.Cu" "B.Cu") (net 1))
@@
   (segment (start 159.004 77.8165) (end 158.6875 77.5) (width 0.8) (layer "B.Cu") (net 1))
   (segment (start 158.6875 90) (end 155.5 90) (width 0.8) (layer "B.Cu") (net 1))
-  (segment (start 180.99 90.75) (end 173 90.75) (width 0.8) (layer "B.Cu") (net 1))
   (segment (start 145 80.5) (end 145 77.8125) (width 0.8) (layer "B.Cu") (net 1))
   (segment (start 159.004 93) (end 159.004 90.3165) (width 0.8) (layer "B.Cu") (net 1))
@@
   (segment (start 155.5 90) (end 152.75 87.25) (width 0.8) (layer "B.Cu") (net 1))
   (segment (start 172.6875 77.5) (end 170 77.5) (width 0.8) (layer "B.Cu") (net 1))
-  (segment (start 184.75 86.99) (end 180.99 90.75) (width 0.8) (layer "B.Cu") (net 1))
   (segment (start 166.5 85.25) (end 164.5 87.25) (width 0.8) (layer "B.Cu") (net 2))
   (segment (start 161.504 90.3085) (end 161.8125 90) (width 0.8) (layer "B.Cu") (net 2))
@@
   (segment (start 178.5 82) (end 177.25 83.25) (width 0.8) (layer "B.Cu") (net 6))
   (segment (start 168.75 87.25) (end 167 89) (width 0.8) (layer "B.Cu") (net 6))
-  (segment (start 165.5 68.5) (end 164.2 67.2) (width 0.8) (layer "B.Cu") (net 27))
-  (segment (start 184.75 71.75) (end 184 71.75) (width 0.8) (layer "B.Cu") (net 27))
-  (segment (start 180.5 70.5) (end 178.5 68.5) (width 0.8) (layer "B.Cu") (net 27))
+  (segment (start 181.75 70.5) (end 180.5 70.5) (width 0.8) (layer "B.Cu") (net 27))
   (segment (start 161.504 65.3085) (end 161.8125 65) (width 0.8) (layer "B.Cu") (net 27))
-  (segment (start 181.75 70.5) (end 180.5 70.5) (width 0.8) (layer "B.Cu") (net 27))
   (segment (start 182.5 71.25) (end 181.75 70.5) (width 0.8) (layer "B.Cu") (net 27))
   (segment (start 161.8125 65) (end 164.2 65) (width 0.8) (layer "B.Cu") (net 27))
   (segment (start 184.25 71.25) (end 182.5 71.25) (width 0.8) (layer "B.Cu") (net 27))
+  (segment (start 165.5 68.5) (end 164.2 67.2) (width 0.8) (layer "B.Cu") (net 27))
+  (segment (start 164.45 65) (end 164.5 64.95) (width 0.8) (layer "B.Cu") (net 27))
   (segment (start 184.75 71.75) (end 184.25 71.25) (width 0.8) (layer "B.Cu") (net 27))
+  (segment (start 161.504 68) (end 161.504 65.3085) (width 0.8) (layer "B.Cu") (net 27))
+  (segment (start 180.5 70.5) (end 178.5 68.5) (width 0.8) (layer "B.Cu") (net 27))
   (segment (start 178.5 68.5) (end 165.5 68.5) (width 0.8) (layer "B.Cu") (net 27))
   (segment (start 164.2 67.2) (end 164.2 65) (width 0.8) (layer "B.Cu") (net 27))
-  (segment (start 164.45 65) (end 164.5 64.95) (width 0.8) (layer "B.Cu") (net 27))
-  (segment (start 161.504 68) (end 161.504 65.3085) (width 0.8) (layer "B.Cu") (net 27))
+  (zone (net 0) (net_name "") (layers F&B.Cu) (hatch edge 0.508)
+    (connect_pads (clearance 0))
+    (min_thickness 0.254)
+    (keepout (tracks allowed) (vias allowed) (pads allowed) (copperpour not_allowed) (footprints allowed))
+    (fill (thermal_gap 0.508) (thermal_bridge_width 0.508))
+    (polygon
+      (pts
+        (xy 190.75 96.25)
+        (xy 183 96.25)
+        (xy 183 89)
+        (xy 190.75 89)
+      )
+    )
+  )
+  (zone (net 0) (net_name "") (layers F&B.Cu) (hatch edge 0.508)
+    (connect_pads (clearance 0))
+    (min_thickness 0.254)
+    (keepout (tracks allowed) (vias allowed) (pads allowed) (copperpour not_allowed) (footprints allowed))
+    (fill (thermal_gap 0.508) (thermal_bridge_width 0.508))
+    (polygon
+      (pts
+        (xy 147 96.25)
+        (xy 138.75 96.25)
+        (xy 138.75 88.5)
+        (xy 147 88.5)
+      )
+    )
+  )
+  (zone (net 0) (net_name "") (layers F&B.Cu) (hatch edge 0.508)
+    (connect_pads (clearance 0))
+    (min_thickness 0.254)
+    (keepout (tracks allowed) (vias allowed) (pads allowed) (copperpour not_allowed) (footprints allowed))
+    (fill (thermal_gap 0.508) (thermal_bridge_width 0.508))
+    (polygon
+      (pts
+        (xy 147 66.75)
+        (xy 138.75 66.75)
+        (xy 138.75 58.5)
+        (xy 147 58.5)
+      )
+    )
+  )
   (zone (net 1) (net_name "GND") (layers F&B.Cu) (hatch edge 0.508)
     (connect_pads (clearance 0.508))
@@
         (xy 190.75 58.5)
       )
+    )
+  )
+  (zone (net 0) (net_name "") (layers F&B.Cu) (hatch edge 0.508)
+    (connect_pads (clearance 0))
+    (min_thickness 0.254)
+    (keepout (tracks allowed) (vias allowed) (pads allowed) (copperpour not_allowed) (footprints allowed))
+    (fill (thermal_gap 0.508) (thermal_bridge_width 0.508))
+    (polygon
+      (pts
+        (xy 190.75 66)
+        (xy 183.25 66)
+        (xy 183.25 58.5)
+        (xy 190.75 58.5)
+      )
